File: keyboard.kicad_pcb (KiCad board)
At the start: 2 copper layers, 431 x 122.3 mm, 453 parts, among them J2 Conn_01x05_Pin, SW1 SW_Push, U1 STM32F072C8Tx, U2 74AHCT1G125, U3 XC6206PxxxMR, U4 USB6B1

Commit message: Made power rails thicker
Routing:
- net GND: track 26.5 -> 16.9 mm
- net Row6: track 747.7 -> 751.7 mm
