File: keyboard.kicad_pcb (KiCad board)
At the start: 2 copper layers, 431 x 122.3 mm, 453 parts, among them J2 Conn_01x05_Pin, SW1 SW_Push, U1 STM32F072C8Tx, U2 74AHCT1G125, U3 XC6206PxxxMR, U4 USB6B1

Commit message: Better LED 5V rail setup and matrix wiring
Connections:
- U1 pad 37: Row1 -> Row6
- U1 pad 38: Row2 -> Row1
- U1 pad 39: Row3 -> Row2
- U1 pad 40: Row4 -> Row3
- U1 pad 41: Row5 -> Row4
- U1 pad 42: Row6 -> Row5
Routing:
- net +5V: track 3115.2 -> 3506.6 mm
- net Row5: track 786.9 -> 452.0 mm
- net Row6: track 751.7 -> 445.3 mm
- net Row4: track 784.5 -> 496.7 mm, vias 2 -> 4
- net Row3: track 827.1 -> 543.3 mm, vias 2 -> 4
- net Row2: track 850.0 -> 571.7 mm, vias 2 -> 4
- net Row1: track 796.0 -> 524.4 mm, vias 2 -> 4
- net Col10: track 253.8 -> 198.3 mm
- net Col09: track 269.2 -> 217.4 mm
- net Col08: track 295.6 -> 245.2 mm
- net Col19: track 206.3 -> 164.1 mm, vias 1 -> 3
- net Col11: track 244.6 -> 202.5 mm
- net Col02: track 450.9 -> 413.3 mm, vias 1 -> 3
- net Col18: track 203.8 -> 168.8 mm, vias 1 -> 3
- net Col01: track 469.9 -> 443.3 mm, vias 1 -> 3
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