File: KeyboardMatrix.kicad_sch (KiCad schematic)
At the start: 210 parts

Commit message: USB differential pair mistake correction. Oh dear. Guess this is the start of Rev 2 now.
Changed lines of the file:
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@@
 	)
 	(hierarchical_label "Col04"
-		(shape input)
+		(shape output)
 		(at 69.85 21.59 90)
 		(effects
@@
 	)
 	(hierarchical_label "Col18"
-		(shape input)
+		(shape output)
 		(at 229.87 21.59 90)
 		(effects
@@
 	)
 	(hierarchical_label "Col01"
-		(shape input)
+		(shape output)
 		(at 35.56 21.59 90)
 		(effects
@@
 	)
 	(hierarchical_label "Col21"
-		(shape input)
+		(shape output)
 		(at 264.16 21.59 90)
 		(effects
@@
 	)
 	(hierarchical_label "Col07"
-		(shape input)
+		(shape output)
 		(at 104.14 21.59 90)
 		(effects
@@
 	)
 	(hierarchical_label "Col15"
-		(shape input)
+		(shape output)
 		(at 195.58 21.59 90)
 		(effects
@@
 	)
 	(hierarchical_label "Col10"
-		(shape input)
+		(shape output)
 		(at 138.43 21.59 90)
 		(effects
@@
 	)
 	(hierarchical_label "Col19"
-		(shape input)
+		(shape output)
 		(at 241.3 21.59 90)
 		(effects
@@
 	)
 	(hierarchical_label "Col20"
-		(shape input)
+		(shape output)
 		(at 252.73 21.59 90)
 		(effects
@@
 	)
 	(hierarchical_label "Col16"
-		(shape input)
+		(shape output)
 		(at 207.01 21.59 90)
 		(effects
@@
 	)
 	(hierarchical_label "Col11"
-		(shape input)
+		(shape output)
 		(at 149.86 21.59 90)
 		(effects
@@
 	)
 	(hierarchical_label "Col02"
-		(shape input)
+		(shape output)
 		(at 46.99 21.59 90)
 		(effects
@@
 	)
 	(hierarchical_label "Col06"
-		(shape input)
+		(shape output)
 		(at 92.71 21.59 90)
 		(effects
@@
 	)
 	(hierarchical_label "Col12"
-		(shape input)
+		(shape output)
 		(at 161.29 21.59 90)
 		(effects
@@
 	)
 	(hierarchical_label "Col05"
-		(shape input)
+		(shape output)
 		(at 81.28 21.59 90)
 		(effects
@@
 	)
 	(hierarchical_label "Col14"
-		(shape input)
+		(shape output)
 		(at 184.15 21.59 90)
 		(effects
@@
 	)
 	(hierarchical_label "Col08"
-		(shape input)
+		(shape output)
 		(at 115.57 21.59 90)
 		(effects
@@
 	)
 	(hierarchical_label "Col17"
-		(shape input)
+		(shape output)
 		(at 218.44 21.59 90)
 		(effects
@@
 	)
 	(hierarchical_label "Col09"
-		(shape input)
+		(shape output)
 		(at 127 21.59 90)
 		(effects
@@
 	)
 	(hierarchical_label "Col13"
-		(shape input)
+		(shape output)
 		(at 172.72 21.59 90)
 		(effects
@@
 	)
 	(hierarchical_label "Col03"
-		(shape input)
+		(shape output)
 		(at 58.42 21.59 90)
 		(effects

Commit message: Revision 2
Changed lines of the file:
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@@
 	)
 	(hierarchical_label "Col04"
-		(shape output)
+		(shape input)
 		(at 69.85 21.59 90)
 		(effects
@@
 	)
 	(hierarchical_label "Col18"
-		(shape output)
+		(shape input)
 		(at 229.87 21.59 90)
 		(effects
@@
 	)
 	(hierarchical_label "Col01"
-		(shape output)
+		(shape input)
 		(at 35.56 21.59 90)
 		(effects
@@
 	)
 	(hierarchical_label "Col21"
-		(shape output)
+		(shape input)
 		(at 264.16 21.59 90)
 		(effects
@@
 	)
 	(hierarchical_label "Col07"
-		(shape output)
+		(shape input)
 		(at 104.14 21.59 90)
 		(effects
@@
 	)
 	(hierarchical_label "Col15"
-		(shape output)
+		(shape input)
 		(at 195.58 21.59 90)
 		(effects
@@
 	)
 	(hierarchical_label "Row5"
-		(shape input)
+		(shape output)
 		(at 30.48 128.27 180)
 		(effects
@@
 	)
 	(hierarchical_label "Col10"
-		(shape output)
+		(shape input)
 		(at 138.43 21.59 90)
 		(effects
@@
 	)
 	(hierarchical_label "Col19"
-		(shape output)
+		(shape input)
 		(at 241.3 21.59 90)
 		(effects
@@
 	)
 	(hierarchical_label "Col20"
-		(shape output)
+		(shape input)
 		(at 252.73 21.59 90)
 		(effects
@@
 	)
 	(hierarchical_label "Col16"
-		(shape output)
+		(shape input)
 		(at 207.01 21.59 90)
 		(effects
@@
 	)
 	(hierarchical_label "Col11"
-		(shape output)
+		(shape input)
 		(at 149.86 21.59 90)
 		(effects
@@
 	)
 	(hierarchical_label "Col02"
-		(shape output)
+		(shape input)
 		(at 46.99 21.59 90)
 		(effects
@@
 	)
 	(hierarchical_label "Col06"
-		(shape output)
+		(shape input)
 		(at 92.71 21.59 90)
 		(effects
@@
 	)
 	(hierarchical_label "Col12"
-		(shape output)
+		(shape input)
 		(at 161.29 21.59 90)
 		(effects
@@
 	)
 	(hierarchical_label "Col05"
-		(shape output)
+		(shape input)
 		(at 81.28 21.59 90)
 		(effects
@@
 	)
 	(hierarchical_label "Col14"
-		(shape output)
+		(shape input)
 		(at 184.15 21.59 90)
 		(effects
@@
 	)
 	(hierarchical_label "Col08"
-		(shape output)
+		(shape input)
 		(at 115.57 21.59 90)
 		(effects
@@
 	)
 	(hierarchical_label "Row3"
-		(shape input)
+		(shape output)
 		(at 30.48 85.09 180)
 		(effects
@@
 	)
 	(hierarchical_label "Col17"
-		(shape output)
+		(shape input)
 		(at 218.44 21.59 90)
 		(effects
@@
 	)
 	(hierarchical_label "Row1"
-		(shape input)
+		(shape output)
 		(at 30.48 41.91 180)
 		(effects
@@
 	)
 	(hierarchical_label "Row6"
-		(shape input)
+		(shape output)
 		(at 30.48 149.86 180)
 		(effects
@@
 	)
 	(hierarchical_label "Row4"
-		(shape input)
+		(shape output)
 		(at 30.48 106.68 180)
 		(effects
@@
 	)
 	(hierarchical_label "Row2"
-		(shape input)
+		(shape output)
 		(at 30.48 63.5 180)
 		(effects
@@
 	)
 	(hierarchical_label "Col09"
-		(shape output)
+		(shape input)
 		(at 127 21.59 90)
 		(effects
@@
 	)
 	(hierarchical_label "Col13"
-		(shape output)
+		(shape input)
 		(at 172.72 21.59 90)
 		(effects
@@
 	)
 	(hierarchical_label "Col03"
-		(shape output)
+		(shape input)
 		(at 58.42 21.59 90)
 		(effects
