File: LEDChain.kicad_sch (KiCad schematic)
At the start: 108 parts

Commit message: Big round of changes. Click to read more.
- Labels on the MCU have been switched around to make routing nicer
- ESD Chip is now right next to the connector
- All 3.3V inputs have the 100nF capacitor correctly placed next to it
    - VDDA has an extra 10uF capacitor (as per the STM32 spec sheet)
    - The start of the 3.3V rail has a 4.7uF capacitor (as per the STM32 spec sheet)
- All LEDs now have a 100nF capacitor connected to it, and a 100ohm resistor at the start of the data line
- LED data line has been level shifted to 5V
Parts:
- added C100, C101, C102, C103, C104, C105, C106, C107, C108, C109, C11, C110, C111, C112, C113, C114, C115, C116, C117, C118, C12, C13, C14, C15, C16, C17, C18, C19, C20, C21, C22, C23, C24, C25, C26, C27, C28, C29, C30, C31, C32, C33, C34, C35, C36, C37, C38, C39, C40, C41, C42, C43, C44, C45, C46, C47, C48, C49, C50, C51, C52, C53, C54, C55, C56, C57, C58, C59, C60, C61, C62, C63, C64, C65, C66, C67, C68, C69, C70, C71, C72, C73, C74, C75, C76, C77, C78, C79, C80, C81, C82, C83, C84, C85, C86, C87, C88, C89, C90, C91, C92, C93, C94, C95, C96, C97, C98, C99: 100nF, Capacitor_SMD:C_0402_1005Metric, symbol Device:C
Connections:
- net +5V: now also C100.2, C101.2, C102.2, C103.2, C104.2, C105.2, C106.2, C107.2, C108.2, C109.2, C11.2, C110.2, C111.2, C112.2, C113.2, C114.2, C115.2, C116.2, C117.2, C118.2, C12.2, C13.2, C14.2, C15.2, C16.2, C17.2, C18.2, C19.2, C20.2, C21.2, C22.2, C23.2, C24.2, C25.2, C26.2, C27.2, C28.2, C29.2, C30.2, C31.2, C32.2, C33.2, C34.2, C35.2, C36.2, C37.2, C38.2, C39.2, C40.2, C41.2, C42.2, C43.2, C44.2, C45.2, C46.2, C47.2, C48.2, C49.2, C50.2, C51.2, C52.2, C53.2, C54.2, C55.2, C56.2, C57.2, C58.2, C59.2, C60.2, C61.2, C62.2, C63.2, C64.2, C65.2, C66.2, C67.2, C68.2, C69.2, C70.2, C71.2, C72.2, C73.2, C74.2, C75.2, C76.2, C77.2, C78.2, C79.2, C80.2, C81.2, C82.2, C83.2, C84.2, C85.2, C86.2, C87.2, C88.2, C89.2, C90.2, C91.2, C92.2, C93.2, C94.2, C95.2, C96.2, C97.2, C98.2, C99.2
- net GND: now also C100.1, C101.1, C102.1, C103.1, C104.1, C105.1, C106.1, C107.1, C108.1, C109.1, C11.1, C110.1, C111.1, C112.1, C113.1, C114.1, C115.1, C116.1, C117.1, C118.1, C12.1, C13.1, C14.1, C15.1, C16.1, C17.1, C18.1, C19.1, C20.1, C21.1, C22.1, C23.1, C24.1, C25.1, C26.1, C27.1, C28.1, C29.1, C30.1, C31.1, C32.1, C33.1, C34.1, C35.1, C36.1, C37.1, C38.1, C39.1, C40.1, C41.1, C42.1, C43.1, C44.1, C45.1, C46.1, C47.1, C48.1, C49.1, C50.1, C51.1, C52.1, C53.1, C54.1, C55.1, C56.1, C57.1, C58.1, C59.1, C60.1, C61.1, C62.1, C63.1, C64.1, C65.1, C66.1, C67.1, C68.1, C69.1, C70.1, C71.1, C72.1, C73.1, C74.1, C75.1, C76.1, C77.1, C78.1, C79.1, C80.1, C81.1, C82.1, C83.1, C84.1, C85.1, C86.1, C87.1, C88.1, C89.1, C90.1, C91.1, C92.1, C93.1, C94.1, C95.1, C96.1, C97.1, C98.1, C99.1
Other:
- moved on the sheet: LED1, LED10, LED100, LED101, LED102, LED103, LED104, LED105, LED106, LED107, LED108, LED11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

Commit message: Keyboard wiring simplifcations + schematic editor warning fixes
Parts:
- LED1, LED10, LED100, LED101, LED102, LED103, LED104, LED105, LED106, LED107, LED108, LED11, LED12, LED13, LED14, LED15, LED16, LED17, LED18, LED19, LED2, LED20, LED21, LED22, LED23, LED24, LED25, LED26, LED27, LED28, LED29, LED3, LED30, LED31, LED32, LED33, LED34, LED35, LED36, LED37, LED38, LED39, LED4, LED40, LED41, LED42, LED43, LED44, LED45, LED46, LED47, LED48, LED49, LED5, LED50, LED51, LED52, LED53, LED54, LED55, LED56, LED57, LED58, LED59, LED6, LED60, LED61, LED62, LED63, LED64, LED65, LED66, LED67, LED68, LED69, LED7, LED70, LED71, LED72, LED73, LED74, LED75, LED76, LED77, LED78, LED79, LED8, LED80, LED81, LED82, LED83, LED84, LED85, LED86, LED87, LED88, LED89, LED9, LED90, LED91, LED92, LED93, LED94, LED95, LED96, LED97, LED98, LED99: symbol marbastlib-various:SK6812MINI-E -> PCM_marbastlib-various:SK6812MINI-E
Connections:
- net +5V: now also C29.1; no longer C29.2
- net GND: now also C29.2; no longer C29.1
- net LED: now also LED19.3 (DIN); no longer LED1.3 (DIN)
- net at LED92.2 (DOUT): now also LED91.3 (DIN); no longer LED93.3 (DIN)
- net at LED92.3 (DIN): now also LED93.2 (DOUT); no longer LED91.2 (DOUT)
- net at LED49.2 (DOUT): now also LED48.3 (DIN); no longer LED50.3 (DIN)
- net at LED49.3 (DIN): now also LED50.2 (DOUT); no longer LED48.2 (DOUT)
- net at LED89.2 (DOUT): now also LED88.3 (DIN); no longer LED90.3 (DIN)
- net at LED89.3 (DIN): now also LED90.2 (DOUT); no longer LED88.2 (DOUT)
- net at LED42.2 (DOUT): now also LED41.3 (DIN); no longer LED43.3 (DIN)
- net at LED42.3 (DIN): now also LED43.2 (DOUT); no longer LED41.2 (DOUT)
- net at LED85.2 (DOUT): now also LED84.3 (DIN); no longer LED86.3 (DIN)
- net at LED85.3 (DIN): now also LED86.2 (DOUT); no longer LED84.2 (DOUT)
- net at LED47.2 (DOUT): now also LED46.3 (DIN); no longer LED48.3 (DIN)
- net at LED47.3 (DIN): now also LED48.2 (DOUT); no longer LED46.2 (DOUT)
- net at LED94.2 (DOUT): now also LED93.3 (DIN); no longer LED95.3 (DIN)
- net at LED94.3 (DIN): now also LED95.2 (DOUT); no longer LED93.2 (DOUT)
- net at LED45.2 (DOUT): now also LED44.3 (DIN); no longer LED46.3 (DIN)
- net at LED83.2 (DOUT): now also LED82.3 (DIN); no longer LED84.3 (DIN)
- net at LED83.3 (DIN): now also LED84.2 (DOUT); no longer LED82.2 (DOUT)
- net at LED3.2 (DOUT): now also LED2.3 (DIN); no longer LED4.3 (DIN)
- net at LED3.3 (DIN): now also LED4.2 (DOUT); no longer LED2.2 (DOUT)
- net at LED52.2 (DOUT): now also LED51.3 (DIN); no longer LED53.3 (DIN)
- net at LED52.3 (DIN): now also LED53.2 (DOUT); no longer LED51.2 (DOUT)
- net at LED8.2 (DOUT): now also LED7.3 (DIN); no longer LED9.3 (DIN)
- net at LED8.3 (DIN): now also LED9.2 (DOUT); no longer LED7.2 (DOUT)
- net at LED45.3 (DIN): now also LED46.2 (DOUT); no longer LED44.2 (DOUT)
- net at LED12.2 (DOUT): now also LED11.3 (DIN); no longer LED13.3 (DIN)
- net at LED12.3 (DIN): now also LED13.2 (DOUT); no longer LED11.2 (DOUT)
- net at LED16.2 (DOUT): now also LED15.3 (DIN); no longer LED17.3 (DIN)
- net at LED16.3 (DIN): now also LED17.2 (DOUT); no longer LED15.2 (DOUT)
- net at LED54.2 (DOUT): now also LED53.3 (DIN); no longer LED55.3 (DIN)
- net at LED54.3 (DIN): now also LED55.2 (DOUT); no longer LED53.2 (DOUT)
- net at LED58.2 (DOUT): now also LED57.3 (DIN); no longer LED59.3 (DIN)
- net at LED58.3 (DIN): now also LED59.2 (DOUT); no longer LED57.2 (DOUT)
- net at LED14.2 (DOUT): now also LED13.3 (DIN); no longer LED15.3 (DIN)
- net at LED14.3 (DIN): now also LED15.2 (DOUT); no longer LED13.2 (DOUT)
- net at LED79.2 (DOUT): now also LED78.3 (DIN); no longer LED80.3 (DIN)
- net at LED79.3 (DIN): now also LED80.2 (DOUT); no longer LED78.2 (DOUT)
- net at LED87.2 (DOUT): now also LED86.3 (DIN); no longer LED88.3 (DIN)
- net at LED87.3 (DIN): now also LED88.2 (DOUT); no longer LED86.2 (DOUT)
- net at LED18.3 (DIN): now also LED19.2 (DOUT); no longer LED17.2 (DOUT)
- net at LED10.2 (DOUT): now also LED9.3 (DIN); no longer LED11.3 (DIN)
- net at LED56.2 (DOUT): now also LED55.3 (DIN); no longer LED57.3 (DIN)
- net at LED1.2 (DOUT): now also LED20.3 (DIN); no longer LED2.3 (DIN)
- net at LED62.3 (DIN): now also LED41.2 (DOUT); no longer LED61.2 (DOUT)
- net at LED96.3 (DIN): now also LED78.2 (DOUT); no longer LED95.2 (DOUT)
- net at LED81.3 (DIN): now also LED82.2 (DOUT); no longer LED80.2 (DOUT)
- net at LED56.3 (DIN): now also LED57.2 (DOUT); no longer LED55.2 (DOUT)
- net at LED81.2 (DOUT): now also LED80.3 (DIN); no longer LED82.3 (DIN)
- net at LED5.3 (DIN): now also LED6.2 (DOUT); no longer LED4.2 (DOUT)
- net at LED77.2 (DOUT): now also LED95.3 (DIN); no longer LED78.3 (DIN)
- net at LED18.2 (DOUT): now also LED17.3 (DIN); no longer LED19.3 (DIN)
- net at LED5.2 (DOUT): now also LED4.3 (DIN); no longer LED6.3 (DIN)
- net at LED60.3 (DIN): now also LED61.2 (DOUT); no longer LED59.2 (DOUT)
- net at LED10.3 (DIN): now also LED11.2 (DOUT); no longer LED9.2 (DOUT)
- net at LED60.2 (DOUT): now also LED59.3 (DIN); no longer LED61.3 (DIN)
- net at LED40.2 (DOUT): now also LED61.3 (DIN); no longer LED41.3 (DIN)
- new net: LED43.3 (DIN), LED44.2 (DOUT)
- new net: LED90.3 (DIN), LED91.2 (DOUT)
- new net: LED1.3 (DIN), LED2.2 (DOUT)
- new net: LED50.3 (DIN), LED51.2 (DOUT)
- new net: LED6.3 (DIN), LED7.2 (DOUT)
Other:
- moved on the sheet: C106, C107, C108, C109, C110, C111, C112, C113, C114, C115, C116, C117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
